Commit message: change model

File: sparrow_description/urdf/vehicle.xacro (robot description, xacro)
@@ -6,8 +6,11 @@
   <link name="base_link">
     <visual>
-      <origin xyz="${vehicle_info['/**']['ros__parameters']['wheel_base']/2.0} 0 0" rpy="${pi/2.0} 0 ${pi}"/>
+      <origin xyz="0.2 0 0.505" rpy="0 0 0"/>
       <geometry>
-        <mesh filename="package://sparrow_description/mesh/lexus.dae" scale="1 1 1"/>
+        <box size="0.72 0.53 1.01"/>
       </geometry>
+      <material name="blue">
+        <color rgba="0 0.746 1 1"/>
+      </material>
     </visual>
   </link>
